Commit message: ur5_IK

File: ur5/models/assets/bullet_data/ur5_description/urdf/ur5_arm.urdf (robot description, URDF)
Before this commit: robot ur5, 11 links, 10 joints
Links:
- removed link base
- removed link tool0
- removed link world
Joints:
- removed joint base_link-base_fixed_joint
- removed joint world_joint
- removed joint wrist_3_link-tool0_fixed_joint
